File: Audio_Interface_rewire.kicad_sch (KiCad schematic)
At the start: 62 parts, among them IC1 REG103GA-3.3_2K5, IC2 PCM2906CDB, IC3 INA849DGKT, J1 USB_B_Micro, J2 SJ-435107RS, J3 Vol. knob1 22k, J4 Vol. knob2 22k, J5 SW_PUSH_3PDT, J6 External mic. conn., Q1 J304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

Commit message: Revert "Finished pcb layout for version 2.0"
This reverts commit 9c98f4441856926bdc06a9c73f1d06339f9013c3. Pushed to wrong branch
Other:
- note added: "HP Mic transisitor"
- note removed: "HP Mic transistor"
Changed lines of the file:
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@@
     (effects (font (size 2 2) (thickness 0.4) bold) (justify left bottom))
   )
-  (text "HP Mic transistor" (at 158.75 96.774 0)
+  (text "HP Mic transisitor" (at 158.75 96.774 0)
     (effects (font (size 2 2) (thickness 0.4) bold) (justify left bottom))
   )
